File: 32u2-breakout.kicad_pcb (KiCad board)
At the start: 2 copper layers, 35.1 x 39.1 mm, 16 parts, among them J1 Conn_01x08_Female, J2 Conn_01x08_Female, J3 Conn_01x04_Female, J4 USB_B_Micro, SW1 SW_DIP_x01, U1 ATmega32U2-AU, Y1 7.3728 MHz

Commit message: Add SPI header, use different crystal
Parts:
- added J5: Conn_02x03_Counter_Clockwise, Connector_PinHeader_2.54mm:PinHeader_2x03_P2.54mm_Vertical, F.Cu at (57.7, 61.2)
- Y1: value 7.3728 MHz -> 16 MHz; footprint Crystal:Crystal_SMD_HC49-SD -> Crystal:Crystal_SMD_SeikoEpson_TSX3225-4Pin_3.2x2.5mm
- moved C2 14.4 mm to (40.6, 47.2), turned to 180 degrees
- moved Y1 5.79 mm to (41.7, 43.7)
- moved C1 3.89 mm to (40.4, 39.9), turned to 180 degrees
Connections:
- Y1 pad 1: Net-(C1-Pad1) -> Net-(C2-Pad1)
- Y1 pad 2: Net-(C2-Pad1) -> Net-(Y1-Pad2)
Routing:
- net Net-(J5-Pad3): track 22.9 -> 43.6 mm, vias 2 -> 3
- net Net-(C2-Pad1): track 19.9 -> 7.58 mm, vias 2 -> 0
- net Net-(J1-Pad3): track 14.0 -> 24.2 mm, vias 0 -> 1
- net Net-(J1-Pad4): track 12.1 -> 18.5 mm, vias 0 -> 1
- net Net-(J1-Pad2): track 16.2 -> 21.3 mm
- net GND: track 18.1 -> 18.8 mm
- net Net-(C1-Pad1): track 13.9 -> 13.3 mm, vias 0 -> 2
Other:
- board text added: "32U2 Breakout Board"

Commit message: Relocate ISP pin header
Parts:
- moved J5 33.1 mm to (35.8, 36.3), turned to 90 degrees
Routing:
- net Net-(J1-Pad3): track 24.2 -> 59.5 mm, vias 1 -> 0
- net Net-(J1-Pad2): track 21.3 -> 52.0 mm, vias 0 -> 2
- net Net-(J1-Pad4): track 18.5 -> 43.2 mm, vias 1 -> 2
- net VCC: track 8.80 -> 12.6 mm
- net Net-(J5-Pad3): track 43.6 -> 41.7 mm, vias 3 -> 5
- net Net-(R2-Pad1): track 20.5 -> 21.6 mm
