File: 32u2-breakout.sch (KiCad schematic (older format))
At the start: 16 parts, among them J1 Conn_01x08_Female, J2 Conn_01x08_Female, J3 Conn_01x04_Female, J4 USB_B_Micro, SW1 SW_DIP_x01, U1 ATmega32U2-AU, Y1 7.3728 MHz

Commit message: Add SPI header, use different crystal
Parts:
- removed Y1: 7.3728 MHz, Crystal:Crystal_SMD_HC49-SD, symbol Device:Crystal
- added J5: Conn_02x03_Counter_Clockwise, Connector_PinHeader_2.54mm:PinHeader_2x03_P2.54mm_Vertical, symbol Connector_Generic:Conn_02x03_Counter_Clockwise
- added Y?: 16 MHz, Crystal:Crystal_SMD_SeikoEpson_TSX3225-4Pin_3.2x2.5mm, symbol Device:Crystal_GND24_Small
- D1: MouserLink https://www.mouser.com/ProductDetail/Inolux/IN-S85ATR?qs=sG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 -> https://www.mouser.com/ProductDetail/Wurth-Electronics/1500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
- R3: MouserLink https://www.mouser.com/ProductDetail/Panasonic/ERJ-U02D2000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 -> https://www.mouser.com/ProductDetail/Yageo/AC0402FR-07200RL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
Connections:
- wire segments 59 -> 75
Changed lines of the file:
@@
 encoding utf-8
 Sheet 1 1
-Title ""
-Date ""
-Rev ""
+Title "32U2 Breakout Board"
+Date "2019-01-08"
+Rev "1.1"
 Comp ""
 Comment1 ""
@@
 	1    0    0    -1
 $EndComp
-$Comp
-L Device:Crystal Y1
-U 1 1 5C2431CB
-P 3050 2250
-F 0 "Y1" V 3004 2381 50  0000 L CNN
-F 1 "7.3728 MHz" V 3095 2381 50  0000 L CNN
-F 2 "Crystal:Crystal_SMD_HC49-SD" H 3050 2250 50  0001 C CNN
-F 3 "~" H 3050 2250 50  0001 C CNN
-F 4 "https://www.mouser.com/ProductDetail/Citizen-FineDevice/HCM4973728000ABJT?qs=sGAEpiMZZMsBj6bBr9Q9abMK2mGYOCsJIHv4t3pryiJvaerj5B6i8A%3d%3d" V 3050 2250 50  0001 C CNN "MouserLink"
-	1    3050 2250
-	0    -1   -1   0
-$EndComp
 Wire Wire Line
 	3050 2100 3850 2100
-Wire Wire Line
-	3050 2400 3700 2400
 Wire Wire Line
 	3700 2400 3700 2300
@@
 $EndComp
 Wire Wire Line
-	2650 2400 3050 2400
-Connection ~ 3050 2400
-Wire Wire Line
 	2450 2400 2250 2400
 Wire Wire Line
@@
 Wire Wire Line
 	3050 2050 3050 2100
-Connection ~ 3050 2100
 Wire Wire Line
 	2450 2050 2250 2050
@@
 	5250 1900 5400 1900
 Wire Wire Line
-	5400 2000 5250 2000
-Wire Wire Line
-	5250 2100 5400 2100
-Wire Wire Line
-	5400 2200 5250 2200
+	5400 2000 5300 2000
+Wire Wire Line
+	5250 2100 5300 2100
+Wire Wire Line
+	5400 2200 5350 2200
 Wire Wire Line
 	5250 2300 5400 2300
@@
 F 2 "LED_SMD:LED_0805_2012Metric" H 5500 4250 50  0001 C CNN
 F 3 "~" H 5500 4250 50  0001 C CNN
-F 4 "https://www.mouser.com/ProductDetail/Inolux/IN-S85ATR?qs=sGAEpiMZZMseGfSY3csMkdgyOOAg6kv232JX8b13KFQasOD4KtBwiA%3d%3d" V 5500 4250 50  0001 C CNN "MouserLink"
+F 4 "https://www.mouser.com/ProductDetail/Wurth-Electronics/150080SS75000?qs=sGAEpiMZZMseGfSY3csMkQ6oANueNQcI%252b2qiSb%2fpwjijcMRPJPia9A%3d%3d" V 5500 4250 50  0001 C CNN "MouserLink"
 	1    5500 4250
 	0    -1   -1   0
@@
 F 2 "Resistor_SMD:R_0402_1005Metric" H 5500 4650 50  0001 C CNN
 F 3 "~" H 5500 4650 50  0001 C CNN
-F 4 "https://www.mouser.com/ProductDetail/Panasonic/ERJ-U02D2000X?qs=sGAEpiMZZMvdGkrng054t1aByN2mwWOc45BdGuhLMFQ%3d" H 5500 4650 50  0001 C CNN "MouserLink"
+F 4 "https://www.mouser.com/ProductDetail/Yageo/AC0402FR-07200RL?qs=sGAEpiMZZMvdGkrng054t2uy2SOblyUPN2Lv4UFEbPE%3d" H 5500 4650 50  0001 C CNN "MouserLink"
 	1    5500 4650
 	1    0    0    -1
@@
 $EndComp
 Wire Wire Line
-	3450 1900 3600 1900
+	3450 1900 3500 1900
 Connection ~ 3600 1900
 Wire Wire Line
@@
 Wire Wire Line
 	2800 1900 2850 1900
+$Comp
+L Connector_Generic:Conn_02x03_Counter_Clockwise J5
+U 1 1 5C355306
+P 6050 1300
+F 0 "J5" H 6100 1617 50  0000 C CNN
+F 1 "Conn_02x03_Counter_Clockwise" H 6100 1526 50  0000 C CNN
+F 2 "Connector_PinHeader_2.54mm:PinHeader_2x03_P2.54mm_Vertical" H 6050 1300 50  0001 C CNN
+F 3 "~" H 6050 1300 50  0001 C CNN
+F 4 "https://www.mouser.com/ProductDetail/Wurth-Electronics/61200621621?qs=sGAEpiMZZMs%252bGHln7q6pm%2fFhW%252btWvhAgbNxkR%252blwXp8Ip%2fAN9J9VOg%3d%3d" H 6050 1300 50  0001 C CNN "MouserLink"
+	1    6050 1300
+	1    0    0    -1
+$EndComp
+Wire Wire Line
+	5850 1300 5300 1300
+Connection ~ 5300 2000
+Wire Wire Line
+	5300 2000 5250 2000
+Wire Wire Line
+	5850 1400 3500 1400
+Connection ~ 3500 1900
+Wire Wire Line
+	3500 1900 3600 1900
+Wire Wire Line
+	3500 1400 3500 1900
+Wire Wire Line
+	5300 1300 5300 2000
+$Comp
+L power:GND #PWR0110
+U 1 1 5C35B311
+P 6350 1400
+F 0 "#PWR0110" H 6350 1150 50  0001 C CNN
+F 1 "GND" V 6355 1272 50  0000 R CNN
+F 2 "" H 6350 1400 50  0001 C CNN
+F 3 "" H 6350 1400 50  0001 C CNN
+	1    6350 1400
+	0    -1   -1   0
+$EndComp
+Wire Wire Line
+	5850 1200 5350 1200
+Wire Wire Line
+	5350 1200 5350 2200
+Connection ~ 5350 2200
+Wire Wire Line
+	5350 2200 5250 2200
+Wire Wire Line
+	6350 1300 6750 1300
+Wire Wire Line
+	6750 1300 6750 2050
+Wire Wire Line
+	6750 2050 5300 2050
+Wire Wire Line
+	5300 2050 5300 2100
+Connection ~ 5300 2100
+Wire Wire Line
+	5300 2100 5400 2100
+$Comp
+L power:VCC #PWR0111
+U 1 1 5C35E179
+P 6350 1200
+F 0 "#PWR0111" H 6350 1050 50  0001 C CNN
+F 1 "VCC" V 6367 1328 50  0000 L CNN
+F 2 "" H 6350 1200 50  0001 C CNN
+F 3 "" H 6350 1200 50  0001 C CNN
+	1    6350 1200
+	0    1    1    0
+$EndComp
+$Comp
+L Device:Crystal_GND24_Small Y?
+U 1 1 5C35EF93
+P 3050 2250
+F 0 "Y?" V 3000 1950 50  0000 L CNN
+F 1 "16 MHz" V 3100 1850 50  0000 L CNN
+F 2 "Crystal:Crystal_SMD_SeikoEpson_TSX3225-4Pin_3.2x2.5mm" H 3050 2250 50  0001 C CNN
+F 3 "~" H 3050 2250 50  0001 C CNN
+	1    3050 2250
+	0    1    1    0
+$EndComp
+Wire Wire Line
+	2650 2400 3050 2400
+Wire Wire Line
+	3050 2100 3050 2150
+Connection ~ 3050 2100
+Wire Wire Line
+	3050 2350 3050 2400
+Connection ~ 3050 2400
+Wire Wire Line
+	3050 2400 3700 2400
 $EndSCHEMATC

Commit message: Relocate ISP pin header
Parts:
- gave numbers to parts that had none: 1
Changed lines of the file:
@@
 $EndComp
 $Comp
-L Device:Crystal_GND24_Small Y?
+L Device:Crystal_GND24_Small Y1
 U 1 1 5C35EF93
 P 3050 2250
-F 0 "Y?" V 3000 1950 50  0000 L CNN
+F 0 "Y1" V 3000 1950 50  0000 L CNN
 F 1 "16 MHz" V 3100 1850 50  0000 L CNN
 F 2 "Crystal:Crystal_SMD_SeikoEpson_TSX3225-4Pin_3.2x2.5mm" H 3050 2250 50  0001 C CNN
